File: famicart/hardware/famicart.kicad_sch (KiCad schematic)
At the start: 35 parts, among them J1 Famicom 60-pin edge, U1 Raspberry Pi Pico 2, U10 74LVC1G17 (M2), U11 74LVC1G08 (/PPUACC), U12 74LVC1G07 (/IRQ), U2 74LVC541 (CPU CTRL), U3 74LVC541 (CPU A8-14), U4 74LVC541 (CPU A0-7), U5 74LVC245 (CPU D), U6 74LVC541 (PPU A8-13), U7 74LVC541 (PPU A0-7), U8 74LVC245 (PPU D), U9 74LVC139

Commit message: famicart rev B: USB-C port, reset switch/header, USB-CDC ROM upload; routed (0 airwires, 0 DRC)
Hardware: USB-C receptacle at the top edge wired to the Pico's USB test points
(TP2/TP3 pads per the Pico 2 datasheet, D+/D- assignment selectable by solder
jumpers, wire pads for hand assembly), CC pull-downs, RUN tactile switch and
RUN/GND header, back-side jumpers. DSN exporter fixes: unique pin ids, NPTH
keepouts, custom-pad extents, front-only placement, fixed pre-routed wires.
Firmware: USB-CDC commands INFO/RESET/BOOTSEL/LOAD/PROFILE with flash
programming of the ROM slot, host tool tools/fcload.py; TinyUSB enabled.

Co-Authored-By: Claude Fable 5.1 <noreply@anthropic.com>
Claude-Session: https://claude.ai/code/session_01RfF2rUHDV6Gz9CaznXPSPp
Parts:
- added J2: RUN/GND (console reset wire), Connector_PinHeader_2.54mm:PinHeader_1x02_P2.54mm_Vertical, symbol Connector_Generic:Conn_01x02
- added J3: USB-C (USB 2.0, HRO TYPE-C-31-M-12), Connector_USB:USB_C_Receptacle_HRO_TYPE-C-31-M-12, symbol Connector:USB_C_Receptacle
- added JP3: USB D+ -> TP_A | TP_B, famicart:SolderJumper-3_P1.6mm_Open, symbol Jumper:SolderJumper_3_Open
- added JP4: USB D- -> TP_B | TP_A, famicart:SolderJumper-3_P1.6mm_Open, symbol Jumper:SolderJumper_3_Open
- added R6, R7: 5.1k, Resistor_SMD:R_0603_1608Metric, symbol Device:R
- added SW1: RESET (RUN), Button_Switch_SMD:SW_SPST_TL3342, symbol Switch:SW_Push
- added W1: TP wire pads (A, B, GND), famicart:WirePads_1x3, symbol famicart:WirePads_1x3
Connections:
- net GND: now also U1.46 (TP1_GND), J2.2 (Pin_2), J3.A1 (GND), J3.A12 (GND), J3.B1 (GND), J3.B12 (GND), J3.S1 (SHIELD), R6.2, R7.2, SW1.2, W1.3 (GND)
- net RUN: now reaches U1.30 (RUN)
- net RUN: now also J2.1 (Pin_1), SW1.1
- net VBUS: now reaches U1.40 (VBUS)
- net VBUS: now also J3.A4 (VBUS), J3.A9 (VBUS), J3.B4 (VBUS), J3.B9 (VBUS)
- new net CC1: J3.A5 (CC1), R6.1
- new net CC2: J3.B5 (CC2), R7.1
- new net USB_DM: J3.A7 (D-), J3.B7 (D-), JP4.2 (C)
- new net USB_DP: J3.A6 (D+), J3.B6 (D+), JP3.2 (C)
- new net USB_TPA: JP3.1 (A), JP4.3 (B), U1.44 (TP_A(USB)), W1.1 (A)
- new net USB_TPB: JP3.3 (B), JP4.1 (A), U1.45 (TP_B(USB)), W1.2 (B)
- no-connect marks 10 -> 18
